Commit message: STL/Launch

File: src/rg_description/urdf/roseguardian.URDF (robot description, URDF)
Before this commit: robot roseguardian, 18 links, 17 joints
Links:
- link base_link: geometry collision mesh filename=package://rg_description/meshes/base_link.STL; visual mesh filename=package://rg_description/meshes/base_link.STL
- link left_back_u: geometry collision mesh filename=package://rg_description/meshes/left_back_u.STL; visual mesh filename=package://rg_description/meshes/left_back_u.STL
- link left_back_wheel: geometry collision mesh filename=package://rg_description/meshes/left_back_wheel.STL; visual mesh filename=package://rg_description/meshes/left_back_wheel.STL
- link left_fron_motor: geometry collision mesh filename=package://rg_description/meshes/left_fron_motor.STL; visual mesh filename=package://rg_description/meshes/left_fron_motor.STL
- link left_fron_wheel: geometry collision mesh filename=package://rg_description/meshes/left_fron_wheel.STL; visual mesh filename=package://rg_description/meshes/left_fron_wheel.STL
- link left_leg: geometry collision mesh filename=package://rg_description/meshes/left_leg.STL; visual mesh filename=package://rg_description/meshes/left_leg.STL
- link right_back_u: geometry collision mesh filename=package://rg_description/meshes/right_back_u.STL; visual mesh filename=package://rg_description/meshes/right_back_u.STL
- link right_back_wheel: geometry collision mesh filename=package://rg_description/meshes/right_back_wheel.STL; visual mesh filename=package://rg_description/meshes/right_back_wheel.STL
- link right_front_motor: geometry collision mesh filename=package://rg_description/meshes/right_front_motor.STL; visual mesh filename=package://rg_description/meshes/right_front_motor.STL
- link right_front_wheel: geometry collision mesh filename=package://rg_description/meshes/right_front_wheel.STL; visual mesh filename=package://rg_description/meshes/right_front_wheel.STL
- link right_leg: geometry collision mesh filename=package://rg_description/meshes/right_leg.STL; visual mesh filename=package://rg_description/meshes/right_leg.STL
- link zed_center: geometry visual mesh filename=package://rg_description/meshes/ZED.stl
